File: kicad/gaggia/gaggia.sch (KiCad schematic (older format))
At the start: 14 parts, among them J1 Screw_Terminal_01x02, J2 Screw_Terminal_01x02, J3 Screw_Terminal_01x02, J4 Conn_01x04_Male, J5 Conn_01x04_Male, J6 Conn_01x04_Male, J7 Conn_01x14_Male, U1 MAX31855KASA, U2 MAX31855KASA, U3 S202S02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

Commit message: Updated schematic
Connections:
- net tft_do is gone; now on net perf_do: U1.5 (SCK), U2.7 (SO)
- net ssr_boiler: now also U7.9 (IO33)
- net ssr_pump: no longer U7.9 (IO33)
- net tft_cs: no longer U1.7 (SO), U2.5 (SCK)
- net temp_brew_cs renamed perf_brew_cs
- net temp_ck renamed perf_ck
- net perf_ck: now also U1.7 (SO), U2.5 (SCK)
- net temp_do renamed perf_do
- net temp_ste_cs renamed perf_ste_cs
Other:
- note added: "Buttons"
- note added: "Temperature Sensors"
- moved on the sheet: J5
Changed lines of the file:
@@
 	1    0    0    -1
 $EndComp
-Text Notes 7900 3450 0    197  ~ 0
+Text Notes 7900 3450 0    100  ~ 0
 Steam
-Text Notes 7950 4800 0    197  ~ 0
+Text Notes 7950 4800 0    100  ~ 0
 Brew
-Text Notes 7900 2300 0    197  ~ 0
+Text Notes 7100 2200 0    100  ~ 0
 Boiler
-Text Notes 7900 1150 0    197  ~ 0
+Text Notes 7100 1050 0    100  ~ 0
 Valve
-Text Notes 7900 1700 0    197  ~ 0
+Text Notes 7100 1600 0    100  ~ 0
 Pump
 $Comp
@@
 L Connector:Conn_01x04_Male J5
 U 1 1 60351F72
-P 4150 2300
-F 0 "J5" H 4300 2550 50  0000 R CNN
-F 1 "Conn_01x04_Male" H 4500 2050 50  0000 R CNN
-F 2 "" H 4150 2300 50  0001 C CNN
-F 3 "~" H 4150 2300 50  0001 C CNN
-	1    4150 2300
+P 3700 2300
+F 0 "J5" H 3850 2550 50  0000 R CNN
+F 1 "Conn_01x04_Male" H 4050 2050 50  0000 R CNN
+F 2 "" H 3700 2300 50  0001 C CNN
+F 3 "~" H 3700 2300 50  0001 C CNN
+	1    3700 2300
 	-1   0    0    -1
 $EndComp
@@
 	1950 1100 1950 900
 Wire Wire Line
-	3950 2500 3300 2500
+	3500 2500 3300 2500
 Wire Wire Line
 	3300 2500 3300 4500
@@
 Text Label 2550 2700 0    50   ~ 0
 dsp_cs
-Text Label 2550 3000 0    50   ~ 0
-temp_ck
-Text Label 2550 2800 0    50   ~ 0
-temp_do
 Wire Wire Line
 	2300 2800 2550 2800
@@
 	2550 3000 2300 3000
 Text Label 7500 3250 0    50   ~ 0
-tft_cs
+perf_ck
 Text Label 7500 3350 0    50   ~ 0
-tft_do
+perf_do
 Wire Wire Line
 	7400 3250 7400 4700
@@
 	7050 4900 7500 4900
 Text Label 7500 4900 0    50   ~ 0
-temp_brew_cs
+perf_brew_cs
 Text Label 7500 3550 0    50   ~ 0
-temp_ste_cs
+perf_ste_cs
 Wire Wire Line
 	2300 4100 2550 4100
 Wire Wire Line
 	2300 3700 2550 3700
-Text Label 2550 3700 0    50   ~ 0
-temp_ste_cs
-Text Label 2550 4100 0    50   ~ 0
-temp_brew_cs
 Wire Wire Line
 	2300 3200 3950 3200
@@
 Text Label 2550 4200 0    50   ~ 0
 ssr_pump
-Text Label 2550 4300 0    50   ~ 0
-ssr_pump
 Text Label 2550 3900 0    50   ~ 0
 ssr_valve
 Wire Wire Line
-	2300 2200 3950 2200
-Wire Wire Line
-	3950 2300 3100 2300
-Wire Wire Line
-	3950 2400 3200 2400
+	2300 2200 3500 2200
+Wire Wire Line
+	3500 2300 3100 2300
+Wire Wire Line
+	3500 2400 3200 2400
 Wire Wire Line
 	3200 2400 3200 4400
+Text Label 2550 4300 0    50   ~ 0
+ssr_boiler
+Text Label 2550 3000 0    50   ~ 0
+perf_ck
+Text Label 2550 2800 0    50   ~ 0
+perf_do
+Text Label 2550 3700 0    50   ~ 0
+perf_ste_cs
+Text Label 2550 4100 0    50   ~ 0
+perf_brew_cs
+Text Notes 7500 2800 2    100  ~ 0
+Temperature Sensors
+Text Notes 4450 3050 2    100  ~ 0
+Buttons
 $EndSCHEMATC
